File: KiCad/index.kicad_pcb (KiCad board)
At the start: 2 copper layers, 64 x 80 mm, 20 parts

Commit message: update schematics and KiCad
Routing:
- net D0: track 67.7 -> 79.6 mm, vias 2 -> 1
- net D2: track 61.9 -> 70.1 mm, vias 1 -> 0
- net DA6: track 30.8 -> 23.7 mm, vias 1 -> 0
- net VCC: track 166.4 -> 172.8 mm, vias 1 -> 0
- net PHI2: track 44.6 -> 38.8 mm, vias 1 -> 0
- net D1: track 61.4 -> 66.7 mm
- net A12: track 37.5 -> 32.3 mm, vias 1 -> 0
- net A2: track 32.5 -> 27.9 mm
- net D5: track 41.6 -> 45.7 mm
- net D4: track 41.6 -> 45.6 mm
- net A6: track 31.7 -> 27.9 mm, vias 1 -> 0
- net A3: track 31.7 -> 27.9 mm, vias 1 -> 0
- net A0: track 41.6 -> 45.1 mm
- net PHI2OUT: track 17.0 -> 20.4 mm
- net D7: track 47.2 -> 50.2 mm, vias 0 -> 2
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Other:
- outline, holes or cut-outs redrawn
